File: sensorOne/hardware/sensorOnePcb/sensorOnePcb.kicad_sch (KiCad schematic)
At the start: 74 parts, among them J1 Conn_01x04_Pin, J2 Screw_Terminal_01x08, J3 Conn_ARM_SWD_TagConnect_TC2030, J4 Conn_01x03_Pin, U1 MSPM0G3507SPTR, U2 MCP2562-H-SN, U3 MAX31856, U4 MAX31856, U5 SPX3819M5-L-5-0, U6 SPX3819M5-L-3-3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

Commit message: PCB cleanup
Parts:
- ADR1, ADR2: now left out of the parts list
- C1, C22, C23, C24, C26, C3, C4, C5: Distributor Link 1 (none) -> https://mou.sr/4dNlwD6; Distributor Link 2 (none) -> https://www.digikey.com/en/products/detail/samsung-electro-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; Field8 (none) -> Basic
- C10, C13, C14, C16, C30, C31, C6, C7, C8, C9: Distributor Link 1 https://mou.sr/4dpIZtL -> https://mou.sr/4nYrB47; Distributor Link 2 https://www.digikey.com/en/products/detail/samsung-electro-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 -> https://www.digikey.com/en/products/detail/yageo/CC0603KRX7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; Field8 (none) -> Basic
- C11, C12, C15, C17: Distributor Link 1 https://mou.sr/4dcPEZy -> https://mou.sr/43Ixhpz; Distributor Link 2 https://www.digikey.com/en/products/detail/samsung-electro-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 -> https://www.digikey.com/en/products/detail/knowles-novacap/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; Field8 (none) -> Basic
- C18, C19: Distributor Link 1 https://mou.sr/3VymwCd -> https://mou.sr/4tXYoaV; Distributor Link 2 (none) -> https://www.digikey.com/en/products/detail/samsung-electro-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; Field8 (none) -> Basic
- C2, C20, C21, C25, C27: Distributor Link 1 (none) -> https://mou.sr/4uLKdaq; Distributor Link 2 (none) -> https://www.digikey.com/en/products/detail/samsung-electro-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; Field8 (none) -> Basic; Manufacturer Samsung -> Samsung Electro-Mechanics
- C28: Distributor Link 1 https://mou.sr/4wKpaWQ -> https://mou.sr/49ZVefG; Distributor Link 2 (none) -> https://www.digikey.com/en/products/detail/samsung-electro-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; Field8 (none) -> Basic
- C29: Distributor Link 1 (none) -> https://mou.sr/49ZVefG; Distributor Link 2 (none) -> https://www.digikey.com/en/products/detail/samsung-electro-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; Field8 (none) -> Basic
- R1, R15, R16, R17, R18: Distributor Link 1 (none) -> https://mou.sr/4dUOUHE; Distributor Link 2 (none) -> https://www.tme.com/us/en-us/details/0603waf0000t5e/smd-res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; Field8 (none) -> Basic
- R10, R12, R13, R5, R6, R9: Distributor Link 1 https://mou.sr/4dA7Paz -> https://mou.sr/4vinUsC; Distributor Link 2 (none) -> https://www.tme.com/us/en-us/details/0603waf1000t5e/smd-res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; Field8 (none) -> Basic
- R11, R14: Distributor Link 1 https://mou.sr/4nCfdXD -> https://mou.sr/4x3bgzy; Distributor Link 2 (none) -> https://www.tme.com/us/en-us/details/0603waf1500t5e/smd-res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; Field8 (none) -> Basic
- R19, R20, R7, R8: Distributor Link 1 https://mou.sr/4df7BXr -> https://mou.sr/4fgJ1qA; Distributor Link 2 (none) -> https://www.tme.com/us/en-us/details/0603waf1002t5e/smd-res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; Field8 (none) -> Basic
- R2, R4: Distributor Link 1 (none) -> https://mou.sr/4nVtD5j; Distributor Link 2 (none) -> https://www.tme.com/us/en-us/details/0603waf5101t5e/smd-res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; Field8 (none) -> Basic
- R21: Distributor Link 1 (none) -> https://mou.sr/4dNJZIl; Distributor Link 2 (none) -> https://www.tme.com/us/en-us/details/0603waf1200t5e/smd-res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; Field8 (none) -> Basic
- R3: Distributor Link 1 (none) -> https://mou.sr/4fQ43MR; Distributor Link 2 (none) -> https://www.digikey.com/en/products/detail/panasonic-indust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; Field8 (none) -> Extended
- U1: Distributor Link 1 https://www.digikey.com/en/products/detail/texas-instrument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 -> https://mou.sr/4akP21Z; Distributor Link 2 https://www.mouser.com/ProductDetail/Texas-Instruments/MSPM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 -> https://www.digikey.com/en/products/detail/texas-instrument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; Field8 (none) -> Extended
- U2: Distributor Link 1 https://www.mouser.com/ProductDetail/Microchip-Technology/M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 -> https://mou.sr/4uKPH56; Distributor Link 2 https://www.digikey.com/en/products/detail/microchip-technology/MCP2562T-H-SN/4079819 -> https://www.digikey.com/en/products/detail/microchip-technology/MCP2562-H-SN/4079836; Field8 (none) -> Extended
- U3, U4: value MAX31856 -> MAX31856MUD+; Distributor Link 1 https://mou.sr/4nzAiBG -> https://mou.sr/3RT1kbw; Distributor Link 2 https://www.digikey.com/en/products/detail/analog-devices-inc-maxim-integrated/MAX31856MUD-/5050138 -> https://www.digikey.com/en/products/detail/analog-devices-inc-maxim-integrated/MAX31856MUD/5050138; Field8 (none) -> Extended
- U5: Distributor Link 1 (none) -> https://mou.sr/49u98qg; Distributor Link 2 (none) -> https://www.digikey.com/en/products/detail/maxlinear-inc/SP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; Field8 (none) -> Extended
- U6: Distributor Link 1 (none) -> https://mou.sr/4dJ23Dm; Distributor Link 2 (none) -> https://www.digikey.com/en/products/detail/maxlinear-inc/SP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; Field8 (none) -> Extended
- U7: Distributor Link 1 https://mou.sr/3Rfpqx5 -> https://mou.sr/4xdHCHU; Distributor Link 2 (none) -> https://www.digikey.com/en/products/detail/stmicroelectroni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; Field8 (none) -> Extended
- X1: Distributor Link 1 https://www.digikey.com/en/products/detail/shenzhen-sctf-el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 -> (none); Distributor Link 2 (none) -> https://www.digikey.com/en/products/detail/shenzhen-sctf-el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; Field8 (none) -> Extended
Other:
- company: (none) -> cavemanSensors
- title: sensorOne Sensor Pod Schematic -> ${boardName} Schematic

Commit message: main connector now 2mm jst, added package details
Parts:
- J1: footprint Connector_PinHeader_2.54mm:PinHeader_1x04_P2.54mm_Vertical -> Connector_JST:JST_PH_B4B-PH-K_1x04_P2.00mm_Vertical; Distributor Link 1 (none) -> https://mou.sr/3PHBmaw; Distributor Link 2 (none) -> https://www.digikey.com/en/products/detail/jst-sales-americ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; Field8 (none) -> Extended; LCSC (none) -> C131334; Manufacturer (none) -> JST; Manufacturer Part Number (none) -> B4B-PH-K-S(LF)(SN); now fitted; now in the parts list
- J2: now not fitted
Changed lines of the file:
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@@
 		(body_style 1)
 		(exclude_from_sim no)
-		(in_bom no)
+		(in_bom yes)
 		(on_board yes)
 		(in_pos_files yes)
-		(dnp yes)
+		(dnp no)
 		(fields_autoplaced yes)
 		(property "Reference" "J1"
@@
 			)
 		)
-		(property "Footprint" "Connector_PinHeader_2.54mm:PinHeader_1x04_P2.54mm_Vertical"
+		(property "Footprint" "Connector_JST:JST_PH_B4B-PH-K_1x04_P2.00mm_Vertical"
 			(at 39.37 185.42 0)
 			(hide yes)
@@
 			)
 		)
-		(property "Datasheet" ""
+		(property "Datasheet" "https://www.jst-mfg.com/product/pdf/eng/ePH.pdf"
 			(at 39.37 185.42 0)
 			(hide yes)
@@
 			)
 		)
-		(property "Description" "Generic connector, single row, 01x04, script generated"
+		(property "Description" "-25℃~+85℃ 1 100V 1x4P 2A 2mm 4 4.5mm 4P 6mm 9.9mm Brass K Pin PA66 PH Through Hole Tin UL94V-0 White 插件,P=2mm Wire To Board Connector ROHS"
 			(at 39.37 185.42 0)
 			(hide yes)
@@
 			)
 		)
+		(property "Distributor Link 1" "https://mou.sr/3PHBmaw"
+			(at 39.37 185.42 0)
+			(hide yes)
+			(show_name no)
+			(do_not_autoplace no)
+			(effects
+				(font
+					(size 1.27 1.27)
+				)
+			)
+		)
+		(property "Distributor Link 2" "https://www.digikey.com/en/products/detail/jst-sales-america-inc/B4B-PH-K-S/926613"
+			(at 39.37 185.42 0)
+			(hide yes)
+			(show_name no)
+			(do_not_autoplace no)
+			(effects
+				(font
+					(size 1.27 1.27)
+				)
+			)
+		)
+		(property "Field8" "Extended"
+			(at 39.37 185.42 0)
+			(hide yes)
+			(show_name no)
+			(do_not_autoplace no)
+			(effects
+				(font
+					(size 1.27 1.27)
+				)
+			)
+		)
+		(property "LCSC" "C131334"
+			(at 39.37 185.42 0)
+			(hide yes)
+			(show_name no)
+			(do_not_autoplace no)
+			(effects
+				(font
+					(size 1.27 1.27)
+				)
+			)
+		)
+		(property "Manufacturer" "JST"
+			(at 39.37 185.42 0)
+			(hide yes)
+			(show_name no)
+			(do_not_autoplace no)
+			(effects
+				(font
+					(size 1.27 1.27)
+				)
+			)
+		)
+		(property "Manufacturer Part Number" "B4B-PH-K-S(LF)(SN)"
+			(at 39.37 185.42 0)
+			(hide yes)
+			(show_name no)
+			(do_not_autoplace no)
+			(effects
+				(font
+					(size 1.27 1.27)
+				)
+			)
+		)
 		(pin "1"
 		)
@@
 		(on_board yes)
 		(in_pos_files yes)
-		(dnp no)
+		(dnp yes)
 		(property "Reference" "J2"
 			(at 397.764 142.24 0)
