File: sensorOne/hardware/sensorOnePcb/sensorOnePcb.kicad_sch (KiCad schematic)
At the start: 74 parts, among them J1 Conn_01x04_Pin, J2 Screw_Terminal_01x08, J3 Conn_ARM_SWD_TagConnect_TC2030, J4 Conn_01x03_Pin, U1 MSPM0G3507SPTR, U2 MCP2562-H-SN, U3 MAX31856MUD+, U4 MAX31856MUD+, U5 SPX3819M5-L-5-0, U6 SPX3819M5-L-3-3, U7 LIS3DH, X1 8M

Commit message: Reorganize monorepo project structure
Parts:
- added U8: ESD2CAN24DCKRQ1, SOT-SC70_3_DCK_TEX, symbol MSPM0L1306TDGS28R:ESD2CAN24DCKRQ1
Connections:
- net CAN+: now also U8.2 (IO)
- net CAN-: now also U8.1 (IO)
- net GND: now also U8.3 (GND)
Other:
- moved on the sheet: C6, C7, J1, R21, R4, U2
